File: OpenRomSwitcher.kicad_pcb (KiCad board)
At the start: 2 copper layers, 19.6 x 43.2 mm, 10 parts, among them J1 CONN_01X04, U1 PLUG, U2 SOCKET

Commit message: Final touches for V1
Other:
- board text added: "Switch"
- board text removed: "Vcc"
Changed lines of the file:
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@@
     (links 41)
     (no_connects 0)
-    (area 147.244999 98.984999 166.953001 142.315001)
+    (area 142.24 88.74 183.11 150.020001)
     (thickness 1.6)
     (drawings 30)
@@
   (title_block
     (title OpenRomSwitcher)
-    (date 2018-01-01)
+    (date 2018-01-07)
     (rev 1)
     (company SukkoPera)
@@
     (39 F.Mask user)
     (44 Edge.Cuts user)
-    (49 F.Fab user hide)
+    (49 F.Fab user)
   )
   (setup
@@
     (visible_elements FFFFFF7F)
     (pcbplotparams
-      (layerselection 0x00030_80000001)
+      (layerselection 0x010f0_80000001)
       (usegerberextensions false)
       (excludeedgelayer true)
@@
       (outputformat 1)
       (mirror false)
-      (drillshape 1)
+      (drillshape 0)
       (scaleselection 1)
-      (outputdirectory ""))
+      (outputdirectory gerbers/))
   )
   (net 0 "")
@@
     (pad 2 smd rect (at 1.35 0 90) (size 1.5 1.3) (layers B.Cu B.Mask)
       (net 5 VCC))
-    (model Resistors_SMD.3dshapes/R_0805.wrl
-      (at (xyz 0 0 0))
-      (scale (xyz 1 1 1))
-      (rotate (xyz 0 0 0))
-    )
   )
   (module Resistors_SMD:R_0805_HandSoldering (layer B.Cu)
@@
     (pad 2 smd rect (at 1.35 0 90) (size 1.5 1.3) (layers B.Cu B.Mask)
       (net 4 "Net-(J1-Pad4)"))
+    (model Resistors_SMD.3dshapes/R_0805.wrl
+      (at (xyz 0 0 0))
+      (scale (xyz 1 1 1))
+      (rotate (xyz 0 0 0))
+    )
   )
   (module OpenRomSwitcher:DIP-28_W15.24mm-Notch locked (layer F.Cu)
@@
   (gr_line (start 161.544 124.46) (end 153.924 124.46) (layer B.SilkS) (width 0.2))
   (gr_line (start 161.544 119.38) (end 161.544 124.46) (layer B.SilkS) (width 0.2))
-  (gr_text Vcc (at 152.654 112.522 90) (layer B.SilkS)
+  (gr_text Switch (at 152.654 112.522 90) (layer B.SilkS)
     (effects (font (size 1 1) (thickness 0.15)) (justify mirror))
   )
